Commit message: SLAM works nicely!

File: urdf/robot.xacro (robot description, xacro)
@@ -89,5 +89,5 @@
   </link>
   <joint name="joint_right_wheel" type="continuous">
-    <origin rpy="0 0 0" xyz="0.2 0.15 -0.03"/>
+    <origin rpy="0 0 0" xyz="0.2 -0.15 -0.03"/>
     <child link="link_right_wheel"/>
     <parent link="link_chassis"/>
@@ -97,5 +97,5 @@
   </joint>
   <joint name="joint_left_wheel" type="continuous">
-    <origin rpy="0 0 0" xyz="0.2 -0.15 -0.03"/>
+    <origin rpy="0 0 0" xyz="0.2 +0.15 -0.03"/>
     <child link="link_left_wheel"/>
     <parent link="link_chassis"/>

Commit message: Path planning needs some tuning

File: urdf/robot.xacro (robot description, xacro)
@@ -166,4 +166,10 @@
     </actuator>
   </transmission>
+  <link name="laser_link"></link>
+  <joint name="laser_joint" type="fixed">
+    <origin xyz="0.251 0 0" rpy="0 0 0"/>
+    <parent link="camera_link"/>
+    <child link="laser_link"/>
+  </joint>
   <link name="link_castor_axis">
     <!-- pose and inertial -->

Commit message: Parameters allow most navigations, BUT, robot gets stuck from time to time => create new robot with round shape!!

File: urdf/robot.xacro (robot description, xacro)
@@ -52,4 +52,5 @@
     <!-- body -->
     <collision name="collision_chassis">
+      <origin rpy="0 0 0" xyz="-0.2 0 0"/>
       <geometry>
         <box size="0.5 0.3 0.07"/>
@@ -57,5 +58,5 @@
     </collision>
     <visual>
-      <origin rpy="0 0 0" xyz="0 0 0"/>
+      <origin rpy="0 0 0" xyz="-0.2 0 0"/>
       <geometry>
         <box size="0.5 0.3 0.07"/>
@@ -89,5 +90,5 @@
   </link>
   <joint name="joint_right_wheel" type="continuous">
-    <origin rpy="0 0 0" xyz="0.2 -0.15 -0.03"/>
+    <origin rpy="0 0 0" xyz="0 -0.15 0"/>
     <child link="link_right_wheel"/>
     <parent link="link_chassis"/>
@@ -97,5 +98,5 @@
   </joint>
   <joint name="joint_left_wheel" type="continuous">
-    <origin rpy="0 0 0" xyz="0.2 +0.15 -0.03"/>
+    <origin rpy="0 0 0" xyz="0 +0.15 0"/>
     <child link="link_left_wheel"/>
     <parent link="link_chassis"/>
@@ -126,5 +127,5 @@
   <joint name="neck_joint" type="fixed">
     <axis xyz="0 1 0" />
-    <origin xyz="0.2 0 0.035" rpy="0 0 0"/>
+    <origin xyz="0 0 0.035" rpy="0 0 0"/>
     <parent link="link_chassis"/>
     <child link="neck_link"/>
@@ -214,5 +215,5 @@
   </joint>
   <joint name="joint_castor_axis" type="continuous">
-    <origin rpy="0 0 0" xyz="-0.25 0 -0.05"/>
+    <origin rpy="0 0 0" xyz="-0.45 0 -0.05"/>
     <child link="link_castor_axis"/>
     <parent link="link_chassis"/>

Commit message: Make Robot symmetric and circular!

File: urdf/robot.xacro (robot description, xacro)
@@ -49,16 +49,16 @@
     <!-- pose and inertial -->
     <pose>0 0 0.1 0 0 0</pose>
-    <xacro:cuboid_inertial mass="10" length="0.5" width="0.3" height="0.07"/>
+    <xacro:cuboid_inertial mass="10" length="0.5" width="0.5" height="0.07"/>
     <!-- body -->
     <collision name="collision_chassis">
-      <origin rpy="0 0 0" xyz="-0.2 0 0"/>
-      <geometry>
-        <box size="0.5 0.3 0.07"/>
-      </geometry>
-    </collision>
-    <visual>
-      <origin rpy="0 0 0" xyz="-0.2 0 0"/>
-      <geometry>
-        <box size="0.5 0.3 0.07"/>
+      <origin rpy="0 0 0" xyz="0 0 0"/>
+      <geometry>
+        <cylinder radius="0.2" length="0.07"/>
+      </geometry>
+    </collision>
+    <visual>
+      <origin rpy="0 0 0" xyz="0 0 0"/>
+      <geometry>
+        <cylinder radius="0.2" length="0.07"/>
       </geometry>
       <material name="blue"/>
@@ -179,14 +179,14 @@
     <!-- body -->
     <collision name="collision_chassis">
+      <origin rpy="0 0 0" xyz="-0.01 0 0"/>
+      <geometry>
+        <box size="0.05 0.035 0.03"/>
+      </geometry>
+    </collision>
+    <visual>
       <origin rpy="0 0 0" xyz="-0.025 0 0"/>
       <geometry>
         <box size="0.05 0.035 0.03"/>
       </geometry>
-    </collision>
-    <visual>
-      <origin rpy="0 0 0" xyz="-0.025 0 0"/>
-      <geometry>
-        <box size="0.05 0.035 0.03"/>
-      </geometry>
     </visual>
   </link>
@@ -207,5 +207,5 @@
   </link>
   <joint name="joint_castor_wheel" type="continuous">
-    <origin rpy="0 0 0" xyz="-0.05 0 -0.015"/>
+    <origin rpy="0 0 0" xyz="-0.03 0 -0.02"/>
     <child link="link_castor_wheel"/>
     <parent link="link_castor_axis"/>
@@ -215,5 +215,5 @@
   </joint>
   <joint name="joint_castor_axis" type="continuous">
-    <origin rpy="0 0 0" xyz="-0.45 0 -0.05"/>
+    <origin rpy="0 0 0" xyz="-0.15 0 -0.05"/>
     <child link="link_castor_axis"/>
     <parent link="link_chassis"/>
@@ -222,3 +222,52 @@
     <joint_properties damping="1.0" friction="1.0"/>
   </joint>
+  <link name="link_castor_axis2">
+    <!-- pose and inertial -->
+    <pose>0 0 0.1 0 0 0</pose>
+    <xacro:cuboid_inertial mass="0.2" length="0.05" width="0.035" height="0.03"/>
+    <!-- body -->
+    <collision name="collision_chassis">
+      <origin rpy="0 0 0" xyz="-0.01 0 0"/>
+      <geometry>
+        <box size="0.05 0.035 0.03"/>
+      </geometry>
+    </collision>
+    <visual>
+      <origin rpy="0 0 0" xyz="-0.025 0 0"/>
+      <geometry>
+        <box size="0.05 0.035 0.03"/>
+      </geometry>
+    </visual>
+  </link>
+  <link name="link_castor_wheel2">
+    <xacro:default_inertial mass="0.2"/>
+    <collision name="link_castor_wheel2_collision">
+      <origin rpy="0 1.5707 1.5707" xyz="0 0 0"/>
+      <geometry>
+        <cylinder length="0.02" radius="0.03"/>
+      </geometry>
+    </collision>
+    <visual name="link_castor_wheel2_visual">
+      <origin rpy="0 1.5707 1.5707" xyz="0 0 0"/>
+      <geometry>
+        <cylinder length="0.02" radius="0.03"/>
+      </geometry>
+    </visual>
+  </link>
+  <joint name="joint_castor_wheel2" type="continuous">
+    <origin rpy="0 0 0" xyz="-0.03 0 -0.02"/>
+    <child link="link_castor_wheel2"/>
+    <parent link="link_castor_axis2"/>
+    <axis rpy="0 0 0" xyz="0 1 0"/>
+    <limit effort="10000" velocity="1000"/>
+    <joint_properties damping="1.0" friction="1.0"/>
+  </joint>
+  <joint name="joint_castor_axis2" type="continuous">
+    <origin rpy="0 0 0" xyz="0.15 0 -0.05"/>
+    <child link="link_castor_axis2"/>
+    <parent link="link_chassis"/>
+    <axis rpy="0 0 0" xyz="0 0 1"/>
+    <limit effort="10000" velocity="1000"/>
+    <joint_properties damping="1.0" friction="1.0"/>
+  </joint>
 </robot>

Commit message: State find basically works

File: urdf/robot.xacro (robot description, xacro)
@@ -131,5 +131,5 @@
     <child link="neck_link"/>
   </joint>
-  <link name="camera_link">
+  <link name="head_link">
     <collision>
       <origin xyz="0 0 0.025" rpy="0 0 0"/>
@@ -149,27 +149,23 @@
     <xacro:cuboid_inertial mass="0.3" length="0.25" width="0.1" height="0.05"/>
   </link>
-  <joint name="camera_joint" type="revolute">
-    <axis xyz="0 0 1" />
+  <joint name="head_joint" type="fixed">
+    <!-- <axis xyz="0 0 1" /> -->
     <origin xyz="0 0 0.1" rpy="0 0 0"/>
     <parent link="neck_link"/>
-    <child link="camera_link"/>
-    <limit effort="10000" velocity="1000" lower="${-pi/4}" upper="${pi/4}"/>
-    <joint_properties damping="1.0" friction="1.0"/>
-  </joint>
-  <transmission name="camera_joint_trans">
-    <type>transmission_interface/SimpleTransmission</type>
-    <joint name="camera_joint">
-      <hardwareInterface>EffortJointInterface</hardwareInterface>
-    </joint>
-    <actuator name="motor1">
-      <hardwareInterface>EffortJointInterface</hardwareInterface>
-      <mechanicalInterface>1</mechanicalInterface>
-    </actuator>
-  </transmission>
+    <child link="head_link"/>
+    <!-- <limit effort="10000" velocity="1000" lower="${-pi/4}" upper="${pi/4}"/> -->
+    <!-- <joint_properties damping="1.0" friction="1.0"/> -->
+  </joint>
   <link name="laser_link"></link>
   <joint name="laser_joint" type="fixed">
     <origin xyz="0.251 0 0" rpy="0 0 0"/>
-    <parent link="camera_link"/>
+    <parent link="head_link"/>
     <child link="laser_link"/>
+  </joint>
+  <link name="camera_link"></link>
+  <joint name="camera_joint" type="fixed">
+    <origin xyz="0.251 0 0" rpy="0 0 0"/>
+    <parent link="head_link"/>
+    <child link="camera_link"/>
   </joint>
   <link name="link_castor_axis">

Commit message: switch to smaller robot

File: urdf/robot.xacro (robot description, xacro)
@@ -2,6 +2,6 @@
 <robot xmlns:xacro="http://www.ros.org/wiki/xacro" name="robot_xacro">
   <xacro:include filename="$(find exp_assignment3_pkg)/urdf/robot.gazebo"/>
-  <xacro:property name="length_wheel" value="0.04" />
-  <xacro:property name="radius_wheel" value="0.1" />
+  <xacro:property name="length_wheel" value="0.02" />
+  <xacro:property name="radius_wheel" value="0.05" />
   <xacro:macro name="default_inertial" params="mass">
     <inertial>
@@ -54,5 +54,5 @@
       <origin rpy="0 0 0" xyz="0 0 0"/>
       <geometry>
-        <cylinder radius="0.2" length="0.07"/>
+        <cylinder radius="0.12" length="0.07"/>
       </geometry>
     </collision>
@@ -60,5 +60,5 @@
       <origin rpy="0 0 0" xyz="0 0 0"/>
       <geometry>
-        <cylinder radius="0.2" length="0.07"/>
+        <cylinder radius="0.15" length="0.07"/>
       </geometry>
       <material name="blue"/>
@@ -90,5 +90,5 @@
   </link>
   <joint name="joint_right_wheel" type="continuous">
-    <origin rpy="0 0 0" xyz="0 -0.15 0"/>
+    <origin rpy="0 0 0" xyz="0 -0.12 -0.05"/>
     <child link="link_right_wheel"/>
     <parent link="link_chassis"/>
@@ -98,5 +98,5 @@
   </joint>
   <joint name="joint_left_wheel" type="continuous">
-    <origin rpy="0 0 0" xyz="0 +0.15 0"/>
+    <origin rpy="0 0 0" xyz="0 +0.12 -0.05"/>
     <child link="link_left_wheel"/>
     <parent link="link_chassis"/>
@@ -211,5 +211,5 @@
   </joint>
   <joint name="joint_castor_axis" type="continuous">
-    <origin rpy="0 0 0" xyz="-0.15 0 -0.05"/>
+    <origin rpy="0 0 0" xyz="-0.12 0 -0.05"/>
     <child link="link_castor_axis"/>
     <parent link="link_chassis"/>
@@ -260,5 +260,5 @@
   </joint>
   <joint name="joint_castor_axis2" type="continuous">
-    <origin rpy="0 0 0" xyz="0.15 0 -0.05"/>
+    <origin rpy="0 0 0" xyz="0.12 0 -0.05"/>
     <child link="link_castor_axis2"/>
     <parent link="link_chassis"/>

Commit message: Improved path planning

File: urdf/robot.xacro (robot description, xacro)
@@ -133,13 +133,13 @@
   <link name="head_link">
     <collision>
-      <origin xyz="0 0 0.025" rpy="0 0 0"/>
-      <geometry>
-        <box size="0.05 0.05 0.05"/>
-      </geometry>
-    </collision>
-    <visual>
-      <origin xyz="0.1 0 0.025" rpy="0 0 0"/>
-      <geometry>
-        <box size="0.25 0.1 0.05"/>
+      <origin xyz="0.03 0 0.025" rpy="0 0 0"/>
+      <geometry>
+        <box size="0.15 0.1 0.05"/>
+      </geometry>
+    </collision>
+    <visual>
+      <origin xyz="0.03 0 0.025" rpy="0 0 0"/>
+      <geometry>
+        <box size="0.15 0.1 0.05"/>
       </geometry>
       <material name="red">
@@ -159,5 +159,5 @@
   <link name="laser_link"></link>
   <joint name="laser_joint" type="fixed">
-    <origin xyz="0.251 0 0" rpy="0 0 0"/>
+    <origin xyz="0.105 0 0" rpy="0 0 0"/>
     <parent link="head_link"/>
     <child link="laser_link"/>
@@ -165,5 +165,5 @@
   <link name="camera_link"></link>
   <joint name="camera_joint" type="fixed">
-    <origin xyz="0.251 0 0" rpy="0 0 0"/>
+    <origin xyz="0.105 0 0" rpy="0 0 0"/>
     <parent link="head_link"/>
     <child link="camera_link"/>

Commit message: Comment, Comment, Comment

File: urdf/robot.xacro (robot description, xacro)
@@ -107,13 +107,13 @@
   <link name="neck_link">
     <collision>
-      <origin xyz="0 0 0.05" rpy="0 0 0"/>
-      <geometry>
-        <cylinder radius="0.04" length="0.1"/>
-      </geometry>
-    </collision>
-    <visual>
-      <origin xyz="0 0 0.05" rpy="0 0 0"/>
-      <geometry>
-        <cylinder radius="0.04" length="0.1"/>
+      <origin xyz="0 0 0.1" rpy="0 0 0"/>
+      <geometry>
+        <cylinder radius="0.01" length="0.25"/>
+      </geometry>
+    </collision>
+    <visual>
+      <origin xyz="0 0 0.1" rpy="0 0 0"/>
+      <geometry>
+        <cylinder radius="0.01" length="0.25"/>
       </geometry>
       <material name="orange"/>
@@ -126,6 +126,5 @@
   </link>
   <joint name="neck_joint" type="fixed">
-    <axis xyz="0 1 0" />
-    <origin xyz="0 0 0.035" rpy="0 0 0"/>
+    <origin xyz="0 0 0.04" rpy="0 -0.785 0"/>
     <parent link="link_chassis"/>
     <child link="neck_link"/>
@@ -133,13 +132,13 @@
   <link name="head_link">
     <collision>
-      <origin xyz="0.03 0 0.025" rpy="0 0 0"/>
-      <geometry>
-        <box size="0.15 0.1 0.05"/>
-      </geometry>
-    </collision>
-    <visual>
-      <origin xyz="0.03 0 0.025" rpy="0 0 0"/>
-      <geometry>
-        <box size="0.15 0.1 0.05"/>
+      <origin xyz="-0.02 0 0.05" rpy="0 0 0"/>
+      <geometry>
+        <box size="0.02 0.1 0.1"/>
+      </geometry>
+    </collision>
+    <visual>
+      <origin xyz="-0.02 0 0.05" rpy="0 0 0"/>
+      <geometry>
+        <box size="0.02 0.1 0.1"/>
       </geometry>
       <material name="red">
@@ -151,5 +150,5 @@
   <joint name="head_joint" type="fixed">
     <!-- <axis xyz="0 0 1" /> -->
-    <origin xyz="0 0 0.1" rpy="0 0 0"/>
+    <origin xyz="0 0 0.2" rpy="0 0.785 0"/>
     <parent link="neck_link"/>
     <child link="head_link"/>
@@ -159,5 +158,5 @@
   <link name="laser_link"></link>
   <joint name="laser_joint" type="fixed">
-    <origin xyz="0.105 0 0" rpy="0 0 0"/>
+    <origin xyz="0.01 0 0" rpy="0 0 0"/>
     <parent link="head_link"/>
     <child link="laser_link"/>
@@ -165,5 +164,5 @@
   <link name="camera_link"></link>
   <joint name="camera_joint" type="fixed">
-    <origin xyz="0.105 0 0" rpy="0 0 0"/>
+    <origin xyz="0.01 0 0" rpy="0 0 0"/>
     <parent link="head_link"/>
     <child link="camera_link"/>
